Commit message: Created calibration software

File: urdf/CTA.urdf (robot description, URDF)
Before this commit: robot CTA, 2 links, 1 joints
Links:
- removed link base_link
- added link cabin_center; visual box size=1.430 2.615 2.256
- added link turret_axis; visual cylinder length=1 radius=1.68
Joints:
- removed joint right_hand_joint
- added joint cebin_center_joint: type fixed, parent turret_axis, child cabin_center, origin xyz=0 0 0 rpy=0 0 0
- added joint cruce_left_joint: type fixed, parent turret_axis, child crucible_left, origin xyz=0 0 0 rpy=0 0 0

Commit message: Attached crucible in both directions

File: urdf/CTA.urdf (robot description, URDF)
Before this commit: robot CTA, 3 links, 2 joints
Links:
- added link crucible_right; visual cylinder length=1.7 radius=1.081
Joints:
- removed joint cebin_center_joint
- added joint cabin_center_joint: type fixed, parent turret_axis, child cabin_center, origin xyz=0 0 0 rpy=0 0 0
- added joint cruce_right_joint: type fixed, parent turret_axis, child crucible_left, origin xyz=0 0 0 rpy=0 0 0

Commit message: Attached crucible in both directions - Fixed

File: urdf/CTA.urdf (robot description, URDF)
Before this commit: robot CTA, 4 links, 3 joints
Joints:
- joint cruce_right_joint: child crucible_left -> crucible_right
